Commit message: add visualisation in gazebo

File: install/ackermann_vehicle_description/share/ackermann_vehicle_description/urdf/car.xacro (robot description, xacro)
@@ -1,6 +1,6 @@
-<?xml version="1.0"?>
 <robot name="car" xmlns:xacro="http://www.ros.org/wiki/xacro">
+  <xacro:property name="pi" value="3.1415926535897931" />
   <xacro:property name="base_width" value="0.4" />
-  <xacro:property name="base_length" value="${base_width * 3.4}" />
+  <xacro:property name="base_length" value="1.36" />
   <xacro:property name="base_height" value="0.6" />
   <xacro:property name="wheel_radius" value="0.20" />
@@ -55,5 +55,5 @@
       <origin xyz="0 0 0.27" rpy="0 0 0"/>
       <geometry>
-        <box size="${base_length + 0.2} ${base_width} ${base_height - 0.2}"/>
+        <box size="1.56 0.4 0.4"/>
       </geometry>
     </collision>
@@ -61,5 +61,5 @@
       <origin xyz="0 0 0" rpy="0 0 0"/>
       <geometry>
-        <mesh filename="file:///home/artem/vechicle/install/ackermann_vehicle_description/share/ackermann_vehicle_description/meshes/car.dae"/>
+        <mesh filename="package://ackermann_vehicle_description/meshes/car.dae"/>
       </geometry>
     </visual>
@@ -69,5 +69,5 @@
     <xacro:if value="${sidefr == 1}">
       <joint name="${suffix}_steering_knuckle_joint" type="revolute">
-        <origin xyz="${base_length / 100 * 35 * sidefr} ${0.4 * sidelr} -0.3" rpy="0 0 ${pi/2}"/>
+        <origin xyz="${0.476 * sidefr} ${0.2 * sidelr} -0.3" rpy="0 0 ${pi/2}"/>
         <parent link="chassis"/>
         <child link="${suffix}_steering_knuckle_link"/>
@@ -78,5 +78,5 @@
     <xacro:unless value="${sidefr == 1}">
       <joint name="${suffix}_steering_knuckle_joint" type="fixed">
-        <origin xyz="${base_length / 100 * 35 * sidefr} ${0.4 * sidelr} -0.3" rpy="0 0 ${pi/2}"/>
+        <origin xyz="${0.476 * sidefr} ${0.2 * sidelr} -0.3" rpy="0 0 ${pi/2}"/>
         <parent link="chassis"/>
         <child link="${suffix}_steering_knuckle_link"/>
@@ -131,5 +131,5 @@
         <origin xyz="0 0 0" rpy="0 ${pi/2} 0"/>
         <geometry>
-          <mesh filename="file:///home/artem/vechicle/install/ackermann_vehicle_description/share/ackermann_vehicle_description/meshes/wheel.dae"/>
+          <mesh filename="package://ackermann_vehicle_description/meshes/wheel.dae"/>
         </geometry>
       </visual>
@@ -142,5 +142,4 @@
   <xacro:wheel suffix="rear_right" sidefr="-1" sidelr="-1" />
   <joint name="hokuyo_joint" type="fixed">
-    <axis xyz="0 0 0" />
     <origin xyz="0.574 0 0.72" rpy="0 0 0"/>
     <parent link="base_link"/>
@@ -157,5 +156,5 @@
       <origin xyz="0 0 0" rpy="0 0 0"/>
       <geometry>
-        <mesh filename="file:///home/artem/vechicle/install/ackermann_vehicle_description/share/ackermann_vehicle_description/meshes/hokuyo.dae"/>
+        <mesh filename="package://ackermann_vehicle_description/meshes/hokuyo.dae"/>
       </geometry>
     </visual>
