Commit message: update visualisation in gazebo

File: ackermann_vehicle_description/urdf/car.xacro (robot description, xacro)
@@ -16,4 +16,19 @@
     <material>CarMaterial</material>
   </gazebo>
+  <material name="Black">
+    <color rgba="0.0 0.0 0.0 1.0"/>
+  </material>
+  <gazebo reference="front_left_wheel_link">
+  <material>Gazebo/Black</material>
+</gazebo>
+<gazebo reference="front_right_wheel_link">
+  <material>Gazebo/Black</material>
+</gazebo>
+<gazebo reference="rear_left_wheel_link">
+  <material>Gazebo/Black</material>
+</gazebo>
+<gazebo reference="rear_right_wheel_link">
+  <material>Gazebo/Black</material>
+</gazebo>
   <xacro:macro name="cylinder_inertial" params="radius height mass">
     <inertial>

Commit message: add lidar + teleop

File: ackermann_vehicle_description/urdf/car.xacro (robot description, xacro)
@@ -20,15 +20,15 @@
   </material>
   <gazebo reference="front_left_wheel_link">
-  <material>Gazebo/Black</material>
-</gazebo>
-<gazebo reference="front_right_wheel_link">
-  <material>Gazebo/Black</material>
-</gazebo>
-<gazebo reference="rear_left_wheel_link">
-  <material>Gazebo/Black</material>
-</gazebo>
-<gazebo reference="rear_right_wheel_link">
-  <material>Gazebo/Black</material>
-</gazebo>
+    <material>Gazebo/Black</material>
+  </gazebo>
+  <gazebo reference="front_right_wheel_link">
+    <material>Gazebo/Black</material>
+  </gazebo>
+  <gazebo reference="rear_left_wheel_link">
+    <material>Gazebo/Black</material>
+  </gazebo>
+  <gazebo reference="rear_right_wheel_link">
+    <material>Gazebo/Black</material>
+  </gazebo>
   <xacro:macro name="cylinder_inertial" params="radius height mass">
     <inertial>
@@ -156,7 +156,8 @@
   <xacro:wheel suffix="rear_left" sidefr="-1" sidelr="1" />
   <xacro:wheel suffix="rear_right" sidefr="-1" sidelr="-1" />
+  <!-- Hokuyo Lidar -->
   <joint name="hokuyo_joint" type="fixed">
     <axis xyz="0 0 0" />
-    <origin xyz="0.574 0 0.72" rpy="0 0 0"/>
+    <origin xyz="0.574 0 0.7" rpy="0 0 0"/>
     <parent link="base_link"/>
     <child link="hokuyo"/>
@@ -176,8 +177,39 @@
     </visual>
     <inertial>
-      <mass value="1e-5" />
-      <origin xyz="0 0 0" rpy="0 0 0"/>
-      <inertia ixx="1e-6" ixy="0" ixz="0" iyy="1e-6" iyz="0" izz="1e-6" />
+      <mass value="0.1" />
+      <origin xyz="0 0 0" rpy="0 0 0"/>
+      <inertia ixx="0.001" ixy="0" ixz="0" iyy="0.001" iyz="0" izz="0.001" />
     </inertial>
   </link>
+  <!-- ============ GAZEBO ЛАЗЕРНЫЙ СКАНЕР ДЛЯ HOKUYO ============ -->
+  <gazebo reference="hokuyo">
+    <sensor name="laser" type="ray">
+      <pose>0 0 0 0 0 0</pose>
+      <visualize>true</visualize>
+      <update_rate>10</update_rate>
+      <ray>
+        <scan>
+          <horizontal>
+            <samples>360</samples>
+            <resolution>1</resolution>
+            <min_angle>-3.14159</min_angle>
+            <max_angle>3.14159</max_angle>
+          </horizontal>
+        </scan>
+        <range>
+          <min>0.9</min>
+          <max>5.0</max>
+          <resolution>0.01</resolution>
+        </range>
+      </ray>
+      <plugin name="laser_plugin" filename="libgazebo_ros_ray_sensor.so">
+        <ros>
+          <namespace>/</namespace>
+          <argument>/scan:=scan</argument>
+        </ros>
+        <output_type>sensor_msgs/LaserScan</output_type>
+        <frame_name>hokuyo</frame_name>
+      </plugin>
+    </sensor>
+  </gazebo>
 </robot>

Commit message: add remote control

File: ackermann_vehicle_description/urdf/car.xacro (robot description, xacro)
@@ -12,11 +12,11 @@
     <color rgba="1.0 1.0 1.0 1.0"/>
   </material>
+  <material name="Black">
+    <color rgba="0.0 0.0 0.0 1.0"/>
+  </material>
   <link name="odom"/>
   <gazebo reference="chassis">
     <material>CarMaterial</material>
   </gazebo>
-  <material name="Black">
-    <color rgba="0.0 0.0 0.0 1.0"/>
-  </material>
   <gazebo reference="front_left_wheel_link">
     <material>Gazebo/Black</material>
@@ -31,21 +31,4 @@
     <material>Gazebo/Black</material>
   </gazebo>
-  <xacro:macro name="cylinder_inertial" params="radius height mass">
-    <inertial>
-      <origin xyz="0 0 0" rpy="0 0 0" />
-      <mass value="${mass}"/>
-      <inertia ixx="${0.5 * mass * radius * radius}"
-               ixy="0" ixz="0"
-               iyy="${0.0833333 * mass * (3 * radius * radius + height * height)}"
-               iyz="0"
-               izz="${0.0833333 * mass * (3 * radius * radius + height * height)}"/>
-    </inertial>
-  </xacro:macro>
-  <xacro:macro name="null_inertial">
-    <inertial>
-      <mass value="0.001"/>
-      <inertia ixx="0.001" ixy="0" ixz="0" iyy="0.001" iyz="0" izz="0.001"/>
-    </inertial>
-  </xacro:macro>
   <link name="base_link">
     <visual>
@@ -79,6 +62,27 @@
       </geometry>
     </visual>
-    <xacro:null_inertial/>
+    <inertial>
+      <mass value="10.0" />
+      <origin xyz="0 0 0" rpy="0 0 0"/>
+      <inertia ixx="1.0" ixy="0" ixz="0" iyy="1.0" iyz="0" izz="1.0" />
+    </inertial>
   </link>
+  <xacro:macro name="cylinder_inertial" params="radius height mass">
+    <inertial>
+      <origin xyz="0 0 0" rpy="0 0 0" />
+      <mass value="${mass}"/>
+      <inertia ixx="${0.5 * mass * radius * radius}"
+               ixy="0" ixz="0"
+               iyy="${0.0833333 * mass * (3 * radius * radius + height * height)}"
+               iyz="0"
+               izz="${0.0833333 * mass * (3 * radius * radius + height * height)}"/>
+    </inertial>
+  </xacro:macro>
+  <xacro:macro name="null_inertial">
+    <inertial>
+      <mass value="0.001"/>
+      <inertia ixx="0.001" ixy="0" ixz="0" iyy="0.001" iyz="0" izz="0.001"/>
+    </inertial>
+  </xacro:macro>
   <xacro:macro name="steering_knuckle" params="suffix sidefr sidelr">
     <xacro:if value="${sidefr == 1}">
@@ -114,22 +118,7 @@
   <xacro:steering_knuckle suffix="rear_right" sidefr="-1" sidelr="-1" />
   <xacro:macro name="wheel" params="suffix sidefr sidelr">
-    <joint name="${suffix}_axel_joint" type="fixed">
+    <joint name="${suffix}_wheel_joint" type="continuous">
       <origin xyz="0 0 0" rpy="0 0 0"/>
       <parent link="${suffix}_steering_knuckle_link"/>
-      <child link="${suffix}_wheel_axel"/>
-    </joint>
-    <link name="${suffix}_wheel_axel">
-      <visual>
-        <origin xyz="0 0 0" rpy="0 0 0"/>
-        <geometry>
-          <sphere radius="0.02" />
-        </geometry>
-        <material name="white"/>
-      </visual>
-      <xacro:null_inertial/>
-    </link>
-    <joint name="${suffix}_wheel_joint" type="continuous">
-      <origin xyz="0 0 0" rpy="0 0 0"/>
-      <parent link="${suffix}_wheel_axel"/>
       <child link="${suffix}_wheel_link"/>
       <axis xyz="1 0 0" />
@@ -213,3 +202,39 @@
     </sensor>
   </gazebo>
+  <!-- ============ GAZEBO ПЛАГИНЫ ДЛЯ УПРАВЛЕНИЯ (ИЗ ВАШЕГО РАБОЧЕГО ПРОЕКТА) ============ -->
+  <gazebo>
+    <plugin name="diff_drive" filename="libgazebo_ros_diff_drive.so">
+      <!-- Wheel Information -->
+      <num_wheel_pairs>2</num_wheel_pairs>
+      <left_joint>rear_left_wheel_joint</left_joint>
+      <left_joint>front_left_wheel_joint</left_joint>
+      <right_joint>rear_right_wheel_joint</right_joint>
+      <right_joint>front_right_wheel_joint</right_joint>
+      <!-- Kinematics -->
+      <wheel_separation>0.4</wheel_separation>
+      <wheel_diameter>0.4</wheel_diameter>
+      <!-- Limits -->
+      <max_wheel_torque>20</max_wheel_torque>
+      <max_wheel_acceleration>2.0</max_wheel_acceleration>
+      <!-- Output -->
+      <odometry_frame>odom</odometry_frame>
+      <robot_base_frame>base_link</robot_base_frame>
+      <publish_odom>true</publish_odom>
+      <publish_odom_tf>true</publish_odom_tf>
+      <publish_wheel_tf>true</publish_wheel_tf>
+      <update_rate>40.0</update_rate>
+    </plugin>
+  </gazebo>
+  <gazebo>
+    <plugin name="diff_drive_joint_states" filename="libgazebo_ros_joint_state_publisher.so">
+      <ros>
+        <remapping>~/out:=joint_states</remapping>
+      </ros>
+      <update_rate>50</update_rate>
+      <left_joint>rear_left_wheel_joint</left_joint>
+      <left_joint>front_left_wheel_joint</left_joint>
+      <right_joint>rear_right_wheel_joint</right_joint>
+      <right_joint>front_right_wheel_joint</right_joint>
+    </plugin>
+  </gazebo>
 </robot>

Commit message: add camera

File: ackermann_vehicle_description/urdf/car.xacro (robot description, xacro)
@@ -238,3 +238,68 @@
     </plugin>
   </gazebo>
+  <joint name="camera_joint" type="fixed">
+    <origin xyz="1.2 0 0.475" rpy="0 0 0"/>
+    <parent link="base_link"/>
+    <child link="camera_link"/>
+  </joint>
+  <link name="camera_link">
+    <!-- Корпус: куб -->
+    <visual>
+      <origin xyz="0 0 0" rpy="0 0 0"/>
+      <geometry>
+        <box size="0.05 0.05 0.05"/>
+      </geometry>
+      <material name="Black"/>
+    </visual>
+    <!-- Объектив: цилиндр -->
+    <visual>
+      <origin xyz="0.035 0 0" rpy="0 1.5708 0"/>
+      <geometry>
+        <cylinder radius="0.02" length="0.03"/>
+      </geometry>
+      <material name="Black"/>
+    </visual>
+    <collision>
+      <origin xyz="0 0 0" rpy="0 0 0"/>
+      <geometry>
+        <box size="0.05 0.05 0.05"/>
+      </geometry>
+    </collision>
+    <inertial>
+      <mass value="0.05"/>
+      <inertia ixx="0.0001" ixy="0" ixz="0" iyy="0.0001" iyz="0" izz="0.0001"/>
+    </inertial>
+  </link>
+  <gazebo reference="camera_link">
+    <material>Gazebo/Black</material>
+    <sensor name="camera" type="camera">
+      <pose>0 0 0 0 0 0</pose>
+      <visualize>true</visualize>
+      <update_rate>30</update_rate>
+      <camera>
+        <horizontal_fov>1.089</horizontal_fov> <!-- 80 градусов -->
+        <image>
+            <format>R8G8B8</format>
+            <width>1920</width>
+            <height>1080</height>
+        </image>
+        <clip>
+          <near>0.5</near>
+          <far>100.0</far>
+        </clip>
+      </camera>
+      <plugin name="camera_controller" filename="libgazebo_ros_camera.so">
+        <ros>
+          <namespace>/</namespace>
+          <argument>/camera/image_raw:=camera/image_raw</argument>
+          <argument>/camera/camera_info:=camera/camera_info</argument>
+        </ros>
+        <camera_name>camera</camera_name>
+        <image_topic_name>image_raw</image_topic_name>
+        <camera_info_topic_name>camera_info</camera_info_topic_name>
+        <frame_name>camera_link</frame_name>
+        <hack_base_name>camera</hack_base_name>
+      </plugin>
+    </sensor>
+  </gazebo>
 </robot>

Commit message: fix lidar + display.launch

File: ackermann_vehicle_description/urdf/car.xacro (robot description, xacro)
@@ -146,11 +146,11 @@
   <xacro:wheel suffix="rear_right" sidefr="-1" sidelr="-1" />
   <!-- Hokuyo Lidar -->
-  <joint name="hokuyo_joint" type="fixed">
+  <joint name="lidar_joint" type="fixed">
     <axis xyz="0 0 0" />
     <origin xyz="0.574 0 0.7" rpy="0 0 0"/>
     <parent link="base_link"/>
-    <child link="hokuyo"/>
+    <child link="lidar_link"/>
   </joint>
-  <link name="hokuyo">
+  <link name="lidar_link">
     <collision>
       <origin xyz="0 0 0" rpy="0 0 0"/>
@@ -172,5 +172,5 @@
   </link>
   <!-- ============ GAZEBO ЛАЗЕРНЫЙ СКАНЕР ДЛЯ HOKUYO ============ -->
-  <gazebo reference="hokuyo">
+  <gazebo reference="lidar_link">
     <sensor name="laser" type="ray">
       <pose>0 0 0 0 0 0</pose>
@@ -198,5 +198,5 @@
         </ros>
         <output_type>sensor_msgs/LaserScan</output_type>
-        <frame_name>hokuyo</frame_name>
+        <frame_name>lidar_link</frame_name>
       </plugin>
     </sensor>

File: install/ackermann_vehicle_description/share/ackermann_vehicle_description/urdf/car.xacro (robot description, xacro)
@@ -1,6 +1,6 @@
+<?xml version="1.0"?>
 <robot name="car" xmlns:xacro="http://www.ros.org/wiki/xacro">
-  <xacro:property name="pi" value="3.1415926535897931" />
   <xacro:property name="base_width" value="0.4" />
-  <xacro:property name="base_length" value="1.36" />
+  <xacro:property name="base_length" value="${base_width * 3.4}" />
   <xacro:property name="base_height" value="0.6" />
   <xacro:property name="wheel_radius" value="0.20" />
@@ -12,25 +12,23 @@
     <color rgba="1.0 1.0 1.0 1.0"/>
   </material>
+  <material name="Black">
+    <color rgba="0.0 0.0 0.0 1.0"/>
+  </material>
   <link name="odom"/>
   <gazebo reference="chassis">
     <material>CarMaterial</material>
   </gazebo>
-  <xacro:macro name="cylinder_inertial" params="radius height mass">
-    <inertial>
-      <origin xyz="0 0 0" rpy="0 0 0" />
-      <mass value="${mass}"/>
-      <inertia ixx="${0.5 * mass * radius * radius}"
-               ixy="0" ixz="0"
-               iyy="${0.0833333 * mass * (3 * radius * radius + height * height)}"
-               iyz="0"
-               izz="${0.0833333 * mass * (3 * radius * radius + height * height)}"/>
-    </inertial>
-  </xacro:macro>
-  <xacro:macro name="null_inertial">
-    <inertial>
-      <mass value="0.001"/>
-      <inertia ixx="0.001" ixy="0" ixz="0" iyy="0.001" iyz="0" izz="0.001"/>
-    </inertial>
-  </xacro:macro>
+  <gazebo reference="front_left_wheel_link">
+    <material>Gazebo/Black</material>
+  </gazebo>
+  <gazebo reference="front_right_wheel_link">
+    <material>Gazebo/Black</material>
+  </gazebo>
+  <gazebo reference="rear_left_wheel_link">
+    <material>Gazebo/Black</material>
+  </gazebo>
+  <gazebo reference="rear_right_wheel_link">
+    <material>Gazebo/Black</material>
+  </gazebo>
   <link name="base_link">
     <visual>
@@ -55,5 +53,5 @@
       <origin xyz="0 0 0.27" rpy="0 0 0"/>
       <geometry>
-        <box size="1.56 0.4 0.4"/>
+        <box size="${base_length + 0.2} ${base_width} ${base_height - 0.2}"/>
       </geometry>
     </collision>
@@ -61,13 +59,34 @@
       <origin xyz="0 0 0" rpy="0 0 0"/>
       <geometry>
-        <mesh filename="package://ackermann_vehicle_description/meshes/car.dae"/>
-      </geometry>
-    </visual>
-    <xacro:null_inertial/>
+        <mesh filename="file:///home/artem/vechicle/install/ackermann_vehicle_description/share/ackermann_vehicle_description/meshes/car.dae"/>
+      </geometry>
+    </visual>
+    <inertial>
+      <mass value="10.0" />
+      <origin xyz="0 0 0" rpy="0 0 0"/>
+      <inertia ixx="1.0" ixy="0" ixz="0" iyy="1.0" iyz="0" izz="1.0" />
+    </inertial>
   </link>
+  <xacro:macro name="cylinder_inertial" params="radius height mass">
+    <inertial>
+      <origin xyz="0 0 0" rpy="0 0 0" />
+      <mass value="${mass}"/>
+      <inertia ixx="${0.5 * mass * radius * radius}"
+               ixy="0" ixz="0"
+               iyy="${0.0833333 * mass * (3 * radius * radius + height * height)}"
+               iyz="0"
+               izz="${0.0833333 * mass * (3 * radius * radius + height * height)}"/>
+    </inertial>
+  </xacro:macro>
+  <xacro:macro name="null_inertial">
+    <inertial>
+      <mass value="0.001"/>
+      <inertia ixx="0.001" ixy="0" ixz="0" iyy="0.001" iyz="0" izz="0.001"/>
+    </inertial>
+  </xacro:macro>
   <xacro:macro name="steering_knuckle" params="suffix sidefr sidelr">
     <xacro:if value="${sidefr == 1}">
       <joint name="${suffix}_steering_knuckle_joint" type="revolute">
-        <origin xyz="${0.476 * sidefr} ${0.2 * sidelr} -0.3" rpy="0 0 ${pi/2}"/>
+        <origin xyz="${base_length / 100 * 35 * sidefr} ${0.4 * sidelr} -0.3" rpy="0 0 ${pi/2}"/>
         <parent link="chassis"/>
         <child link="${suffix}_steering_knuckle_link"/>
@@ -78,5 +97,5 @@
     <xacro:unless value="${sidefr == 1}">
       <joint name="${suffix}_steering_knuckle_joint" type="fixed">
-        <origin xyz="${0.476 * sidefr} ${0.2 * sidelr} -0.3" rpy="0 0 ${pi/2}"/>
+        <origin xyz="${base_length / 100 * 35 * sidefr} ${0.4 * sidelr} -0.3" rpy="0 0 ${pi/2}"/>
         <parent link="chassis"/>
         <child link="${suffix}_steering_knuckle_link"/>
@@ -99,22 +118,7 @@
   <xacro:steering_knuckle suffix="rear_right" sidefr="-1" sidelr="-1" />
   <xacro:macro name="wheel" params="suffix sidefr sidelr">
-    <joint name="${suffix}_axel_joint" type="fixed">
+    <joint name="${suffix}_wheel_joint" type="continuous">
       <origin xyz="0 0 0" rpy="0 0 0"/>
       <parent link="${suffix}_steering_knuckle_link"/>
-      <child link="${suffix}_wheel_axel"/>
-    </joint>
-    <link name="${suffix}_wheel_axel">
-      <visual>
-        <origin xyz="0 0 0" rpy="0 0 0"/>
-        <geometry>
-          <sphere radius="0.02" />
-        </geometry>
-        <material name="white"/>
-      </visual>
-      <xacro:null_inertial/>
-    </link>
-    <joint name="${suffix}_wheel_joint" type="continuous">
-      <origin xyz="0 0 0" rpy="0 0 0"/>
-      <parent link="${suffix}_wheel_axel"/>
       <child link="${suffix}_wheel_link"/>
       <axis xyz="1 0 0" />
@@ -131,5 +135,5 @@
         <origin xyz="0 0 0" rpy="0 ${pi/2} 0"/>
         <geometry>
-          <mesh filename="package://ackermann_vehicle_description/meshes/wheel.dae"/>
+          <mesh filename="file:///home/artem/vechicle/install/ackermann_vehicle_description/share/ackermann_vehicle_description/meshes/wheel.dae"/>
         </geometry>
       </visual>
@@ -141,6 +145,8 @@
   <xacro:wheel suffix="rear_left" sidefr="-1" sidelr="1" />
   <xacro:wheel suffix="rear_right" sidefr="-1" sidelr="-1" />
+  <!-- Hokuyo Lidar -->
   <joint name="hokuyo_joint" type="fixed">
-    <origin xyz="0.574 0 0.72" rpy="0 0 0"/>
+    <axis xyz="0 0 0" />
+    <origin xyz="0.574 0 0.7" rpy="0 0 0"/>
     <parent link="base_link"/>
     <child link="hokuyo"/>
@@ -156,12 +162,144 @@
       <origin xyz="0 0 0" rpy="0 0 0"/>
       <geometry>
-        <mesh filename="package://ackermann_vehicle_description/meshes/hokuyo.dae"/>
-      </geometry>
-    </visual>
-    <inertial>
-      <mass value="1e-5" />
-      <origin xyz="0 0 0" rpy="0 0 0"/>
-      <inertia ixx="1e-6" ixy="0" ixz="0" iyy="1e-6" iyz="0" izz="1e-6" />
+        <mesh filename="file:///home/artem/vechicle/install/ackermann_vehicle_description/share/ackermann_vehicle_description/meshes/hokuyo.dae"/>
+      </geometry>
+    </visual>
+    <inertial>
+      <mass value="0.1" />
+      <origin xyz="0 0 0" rpy="0 0 0"/>
+      <inertia ixx="0.001" ixy="0" ixz="0" iyy="0.001" iyz="0" izz="0.001" />
     </inertial>
   </link>
+  <!-- ============ GAZEBO ЛАЗЕРНЫЙ СКАНЕР ДЛЯ HOKUYO ============ -->
+  <gazebo reference="hokuyo">
+    <sensor name="laser" type="ray">
+      <pose>0 0 0 0 0 0</pose>
+      <visualize>true</visualize>
+      <update_rate>10</update_rate>
+      <ray>
+        <scan>
+          <horizontal>
+            <samples>360</samples>
+            <resolution>1</resolution>
+            <min_angle>-3.14159</min_angle>
+            <max_angle>3.14159</max_angle>
+          </horizontal>
+        </scan>
+        <range>
+          <min>0.9</min>
+          <max>5.0</max>
+          <resolution>0.01</resolution>
+        </range>
+      </ray>
+      <plugin name="laser_plugin" filename="libgazebo_ros_ray_sensor.so">
+        <ros>
+          <namespace>/</namespace>
+          <argument>/scan:=scan</argument>
+        </ros>
+        <output_type>sensor_msgs/LaserScan</output_type>
+        <frame_name>hokuyo</frame_name>
+      </plugin>
+    </sensor>
+  </gazebo>
+  <!-- ============ GAZEBO ПЛАГИНЫ ДЛЯ УПРАВЛЕНИЯ (ИЗ ВАШЕГО РАБОЧЕГО ПРОЕКТА) ============ -->
+  <gazebo>
+    <plugin name="diff_drive" filename="libgazebo_ros_diff_drive.so">
+      <!-- Wheel Information -->
+      <num_wheel_pairs>2</num_wheel_pairs>
+      <left_joint>rear_left_wheel_joint</left_joint>
+      <left_joint>front_left_wheel_joint</left_joint>
+      <right_joint>rear_right_wheel_joint</right_joint>
+      <right_joint>front_right_wheel_joint</right_joint>
+      <!-- Kinematics -->
+      <wheel_separation>0.4</wheel_separation>
+      <wheel_diameter>0.4</wheel_diameter>
+      <!-- Limits -->
+      <max_wheel_torque>20</max_wheel_torque>
+      <max_wheel_acceleration>2.0</max_wheel_acceleration>
+      <!-- Output -->
+      <odometry_frame>odom</odometry_frame>
+      <robot_base_frame>base_link</robot_base_frame>
+      <publish_odom>true</publish_odom>
+      <publish_odom_tf>true</publish_odom_tf>
+      <publish_wheel_tf>true</publish_wheel_tf>
+      <update_rate>40.0</update_rate>
+    </plugin>
+  </gazebo>
+  <gazebo>
+    <plugin name="diff_drive_joint_states" filename="libgazebo_ros_joint_state_publisher.so">
+      <ros>
+        <remapping>~/out:=joint_states</remapping>
+      </ros>
+      <update_rate>50</update_rate>
+      <left_joint>rear_left_wheel_joint</left_joint>
+      <left_joint>front_left_wheel_joint</left_joint>
+      <right_joint>rear_right_wheel_joint</right_joint>
+      <right_joint>front_right_wheel_joint</right_joint>
+    </plugin>
+  </gazebo>
+  <joint name="camera_joint" type="fixed">
+    <origin xyz="1.2 0 0.475" rpy="0 0 0"/>
+    <parent link="base_link"/>
+    <child link="camera_link"/>
+  </joint>
+  <link name="camera_link">
+    <!-- Корпус: куб -->
+    <visual>
+      <origin xyz="0 0 0" rpy="0 0 0"/>
+      <geometry>
+        <box size="0.05 0.05 0.05"/>
+      </geometry>
+      <material name="Black"/>
+    </visual>
+    <!-- Объектив: цилиндр -->
+    <visual>
+      <origin xyz="0.035 0 0" rpy="0 1.5708 0"/>
+      <geometry>
+        <cylinder radius="0.02" length="0.03"/>
+      </geometry>
+      <material name="Black"/>
+    </visual>
+    <collision>
+      <origin xyz="0 0 0" rpy="0 0 0"/>
+      <geometry>
+        <box size="0.05 0.05 0.05"/>
+      </geometry>
+    </collision>
+    <inertial>
+      <mass value="0.05"/>
+      <inertia ixx="0.0001" ixy="0" ixz="0" iyy="0.0001" iyz="0" izz="0.0001"/>
+    </inertial>
+  </link>
+  <gazebo reference="camera_link">
+    <material>Gazebo/Black</material>
+    <sensor name="camera" type="camera">
+      <pose>0 0 0 0 0 0</pose>
+      <visualize>true</visualize>
+      <update_rate>30</update_rate>
+      <camera>
+        <horizontal_fov>1.089</horizontal_fov> <!-- 80 градусов -->
+        <image>
+            <format>R8G8B8</format>
+            <width>1920</width>
+            <height>1080</height>
+        </image>
+        <clip>
+          <near>0.5</near>
+          <far>100.0</far>
+        </clip>
+      </camera>
+      <plugin name="camera_controller" filename="libgazebo_ros_camera.so">
+        <ros>
+          <namespace>/</namespace>
+          <argument>/camera/image_raw:=camera/image_raw</argument>
+          <argument>/camera/camera_info:=camera/camera_info</argument>
+        </ros>
+        <camera_name>camera</camera_name>
+        <image_topic_name>image_raw</image_topic_name>
+        <camera_info_topic_name>camera_info</camera_info_topic_name>
+        <frame_name>camera_link</frame_name>
+        <hack_base_name>camera</hack_base_name>
+      </plugin>
+    </sensor>
+  </gazebo>
 </robot>
